Commit message: replace base_link by torso_base_link within urdf and sdrf

File: motoman_sda10f_support/urdf/sda10f.xacro (robot description, xacro)
@@ -4,9 +4,9 @@
   <joint name="world_joint" type="fixed">
     <parent link="world" />
-    <child link = "base_link" />
+    <child link = "torso_base_link" />
     <origin xyz="0.0 0.0 0.0" rpy="0.0 0.0 0.0" />
   </joint>
   <xacro:include filename="$(find motoman_sda10f_support)/urdf/sda10f_macro.xacro" />
-  <!-- <xacro:motoman_sda10f prefix=""/> -->
+  <xacro:motoman_sda10f prefix=""/>
   <xacro:include filename="$(find motoman_sda10f_support)/urdf/sda10f_transmission.xacro"/>
   <xacro:include filename="$(find motoman_sda10f_support)/urdf/gazebo_plugin.xacro"/>
