Commit message: fix arm xacro with correct prefix

File: motoman_sda10f_support/urdf/sda10f_joint_limited.xacro (robot description, xacro)
@@ -4,9 +4,9 @@
   <joint name="world_joint" type="fixed">
     <parent link="world" />
-    <child link = "base_link" />
+    <child link = "torso_base_link" />
     <origin xyz="0.0 0.0 0.0" rpy="0.0 0.0 0.0" />
   </joint>
   <xacro:include filename="$(find motoman_sda10f_support)/urdf/sda10f_joint_limited_macro.xacro" />
-  <!-- <xacro:motoman_sda10f prefix=""/> -->
+  <xacro:motoman_sda10f prefix=""/>
   <xacro:include filename="$(find motoman_sda10f_support)/urdf/sda10f_transmission.xacro"/>
   <xacro:include filename="$(find motoman_sda10f_support)/urdf/gazebo_plugin.xacro"/>

File: motoman_sda10f_support/urdf/sda10f_joint_limited_macro.xacro (robot description, xacro)
@@ -1,31 +1,35 @@
 <?xml version="1.0" ?>
-<robot xmlns:xacro="http://ros.org/wiki/xacro"
-    name="sda10f">
+<robot xmlns:xacro="http://ros.org/wiki/xacro">
         <xacro:include filename="$(find motoman_sda10f_support)/urdf/common_torso_macro.xacro" />
         <xacro:include filename="$(find motoman_sda10f_support)/urdf/arm_macro.xacro" />
-        <xacro:torso name="torso" prefix="torso_"/>
-        <xacro:motoman_arm name="arm_left" prefix="arm_left_" parent="torso_link_b1" reflect="1"
-             joint_limited="true"
-             link_1_s_lower_limit="${-pi}"  link_1_s_upper_limit="${pi}"
-             link_2_l_lower_limit="${-pi}"  link_2_l_upper_limit="${pi}"
-             link_3_e_lower_limit="${-pi}"  link_3_e_upper_limit="${pi}"
-             link_4_u_lower_limit="${-pi}"  link_4_u_upper_limit="${pi}"
-             link_5_r_lower_limit="${-pi}"  link_5_r_upper_limit="${pi}"
-             link_6_b_lower_limit="${-pi}"  link_6_b_upper_limit="${pi}"
-             link_7_t_lower_limit="${-pi}"  link_7_t_upper_limit="${pi}"
-             >
-            <origin xyz="0.09996 0.0275 0.32214" rpy="1.57 0 0" />
-        </xacro:motoman_arm>
-        <xacro:motoman_arm name="arm_right" prefix="arm_right_" parent="torso_link_b1" reflect="-1"
-            joint_limited="true"
-            link_1_s_lower_limit="${-pi}"  link_1_s_upper_limit="${pi}"
-            link_2_l_lower_limit="${-pi}"  link_2_l_upper_limit="${pi}"
-            link_3_e_lower_limit="${-pi}"  link_3_e_upper_limit="${pi}"
-            link_4_u_lower_limit="${-pi}"  link_4_u_upper_limit="${pi}"
-            link_5_r_lower_limit="${-pi}"  link_5_r_upper_limit="${pi}"
-            link_6_b_lower_limit="${-pi}"  link_6_b_upper_limit="${pi}"
-            link_7_t_lower_limit="${-pi}"  link_7_t_upper_limit="${pi}"
-            >
-            <origin xyz="0.09996 -0.0275 0.32214" rpy="1.57 0 0" />
-        </xacro:motoman_arm>
+        <xacro:macro name="motoman_sda10f" params="prefix">
+            <xacro:torso name="${prefix}torso" prefix="${prefix}torso_"/>
+            <xacro:motoman_arm name="${prefix}arm_left" prefix="${prefix}arm_left_" parent="${prefix}torso_link_b1" reflect="1"
+                 joint_limited="true"
+                 link_1_s_lower_limit="${-pi}"  link_1_s_upper_limit="${pi}"
+                 link_2_l_lower_limit="${-pi}"  link_2_l_upper_limit="${pi}"
+                 link_3_e_lower_limit="${-pi}"  link_3_e_upper_limit="${pi}"
+                 link_4_u_lower_limit="${-pi}"  link_4_u_upper_limit="${pi}"
+                 link_5_r_lower_limit="${-pi}"  link_5_r_upper_limit="${pi}"
+                 link_6_b_lower_limit="${-pi}"  link_6_b_upper_limit="${pi}"
+                 link_7_t_lower_limit="${-pi}"  link_7_t_upper_limit="${pi}"
+                 >
+                <origin xyz="0.09996 0.0275 0.32214" rpy="1.57 0 0" />
+            </xacro:motoman_arm>
+            <xacro:motoman_arm name="${prefix}arm_right" prefix="${prefix}arm_right_" parent="${prefix}torso_link_b1" reflect="-1"
+                joint_limited="true"
+                link_1_s_lower_limit="${-pi}"  link_1_s_upper_limit="${pi}"
+                link_2_l_lower_limit="${-pi}"  link_2_l_upper_limit="${pi}"
+                link_3_e_lower_limit="${-pi}"  link_3_e_upper_limit="${pi}"
+                link_4_u_lower_limit="${-pi}"  link_4_u_upper_limit="${pi}"
+                link_5_r_lower_limit="${-pi}"  link_5_r_upper_limit="${pi}"
+                link_6_b_lower_limit="${-pi}"  link_6_b_upper_limit="${pi}"
+                link_7_t_lower_limit="${-pi}"  link_7_t_upper_limit="${pi}"
+                >
+                <origin xyz="0.09996 -0.0275 0.32214" rpy="1.57 0 0" />
+            </xacro:motoman_arm>
+        </xacro:macro>
+        <xacro:macro name="sda10f">
+            <xacro:motoman_sda10f prefix=""/>
+        </xacro:macro>
 </robot>
