Commit message: Barely working gazebo simulation of SDA10. Lot's of ugly stuff, DO CLEANUP PLEASE.

File: motoman_sda10f_support/urdf/arm_macro.xacro (robot description, xacro)
@@ -19,4 +19,10 @@
 				<material name="yellow"/>
 			</collision>
+	    <inertial>
+	      <mass value="1" />
+	      <inertia ixx="1.0" ixy="0.0" ixz="0.0"
+	               iyy="1.0" iyz="0.0"
+	               izz="1.0" />
+	    </inertial>
 		</link>
 		<link name="${prefix}link_2_l">
@@ -35,4 +41,10 @@
 				<material name="yellow"/>
 			</collision>
+	    <inertial>
+	      <mass value="1" />
+	      <inertia ixx="1.0" ixy="0.0" ixz="0.0"
+	               iyy="1.0" iyz="0.0"
+	               izz="1.0" />
+	    </inertial>
 		</link>
 		<link name="${prefix}link_3_e">
@@ -51,4 +63,10 @@
 				<material name="yellow"/>
 			</collision>
+	    <inertial>
+	      <mass value="1" />
+	      <inertia ixx="1.0" ixy="0.0" ixz="0.0"
+	               iyy="1.0" iyz="0.0"
+	               izz="1.0" />
+	    </inertial>
 		</link>
 		<link name="${prefix}link_4_u">
@@ -67,4 +85,10 @@
 				<material name="yellow"/>
 			</collision>
+	    <inertial>
+	      <mass value="1" />
+	      <inertia ixx="1.0" ixy="0.0" ixz="0.0"
+	               iyy="1.0" iyz="0.0"
+	               izz="1.0" />
+	    </inertial>
 		</link>
 		<link name="${prefix}link_5_r">
@@ -83,4 +107,10 @@
 				<material name="yellow"/>
 			</collision>
+	    <inertial>
+	      <mass value="1" />
+	      <inertia ixx="1.0" ixy="0.0" ixz="0.0"
+	               iyy="1.0" iyz="0.0"
+	               izz="1.0" />
+	    </inertial>
 		</link>
 		<link name="${prefix}link_6_b">
@@ -99,4 +129,10 @@
 				<material name="yellow"/>
 			</collision>
+	    <inertial>
+	      <mass value="1" />
+	      <inertia ixx="1.0" ixy="0.0" ixz="0.0"
+	               iyy="1.0" iyz="0.0"
+	               izz="1.0" />
+	    </inertial>
 		</link>
 		<link name="${prefix}link_7_t">
@@ -113,6 +149,19 @@
 				<material name="yellow"/>
 			</collision>
-		</link>
-	    <link name="${prefix}link_tool0" />
+	    <inertial>
+	      <mass value="1" />
+	      <inertia ixx="1.0" ixy="0.0" ixz="0.0"
+	               iyy="1.0" iyz="0.0"
+	               izz="1.0" />
+	    </inertial>
+		</link>
+	    <link name="${prefix}link_tool0" >
+	    <inertial>
+	      <mass value="1" />
+	      <inertia ixx="1.0" ixy="0.0" ixz="0.0"
+	               iyy="1.0" iyz="0.0"
+	               izz="1.0" />
+	    </inertial>
+</link>
 		<joint name="${prefix}joint_1_s" type="revolute">
 			<parent link="torso_link_b1"/>

File: motoman_sda10f_support/urdf/common_torso_macro.xacro (robot description, xacro)
@@ -20,4 +20,10 @@
 				</material>
 			</collision>
+	    <inertial>
+	      <mass value="1" />
+	      <inertia ixx="1.0" ixy="0.0" ixz="0.0"
+	               iyy="1.0" iyz="0.0"
+	               izz="1.0" />
+	    </inertial>
 		</link>
 		<link name="${prefix}link_b1">
@@ -38,6 +44,12 @@
 				<material name="yellow"/>
 			</collision>
+	    <inertial>
+	      <mass value="1" />
+	      <inertia ixx="1.0" ixy="0.0" ixz="0.0"
+	               iyy="1.0" iyz="0.0"
+	               izz="1.0" />
+	    </inertial>
 		</link>
-		<link name="${prefix}link_b2">
+<!-- 		<link name="${prefix}link_b2">
 			<visual>
 				<origin rpy="0 0 0" xyz="0 0 0"/>
@@ -56,5 +68,11 @@
 				<material name="yellow"/>
 			</collision>
-		</link>
+	    <inertial>
+	      <mass value="1" />
+	      <inertia ixx="1.0" ixy="0.0" ixz="0.0"
+	               iyy="1.0" iyz="0.0"
+	               izz="1.0" />
+	    </inertial>
+		</link> -->
 		<!-- joint list -->
 		<joint name="${prefix}joint_b1" type="revolute">
@@ -65,5 +83,5 @@
 			<limit lower="-2.9570" upper="2.9570" effort="100" velocity="2.26" />
 		</joint>
-		<joint name="${prefix}joint_b2" type="revolute">
+<!-- 		<joint name="${prefix}joint_b2" type="revolute">
 			<parent link="base_link"/>
 			<child link="${prefix}link_b2"/>
@@ -72,5 +90,5 @@
 			<limit lower="-2.9570" upper="2.9570" effort="100" velocity="2.26" />
 			<mimic joint="${prefix}joint_b1" multiplier="1" offset="0"/>
-		</joint>
+		</joint> -->
 		<!-- end of joint list -->
 	</xacro:macro>

File: motoman_sda10f_support/urdf/sda10f.xacro (robot description, xacro)
@@ -1,5 +1,13 @@
 <?xml version="1.0" ?>
 <robot name="motoman_sda10f" xmlns:xacro="http://ros.org/wiki/xacro">
-	<xacro:include filename="$(find motoman_sda10f_support)/urdf/sda10f_macro.xacro" />
-	<xacro:motoman_sda10f prefix=""/>
+  <link name="world"/>
+  <joint name="world_joint" type="fixed">
+    <parent link="world" />
+    <child link = "base_link" />
+    <origin xyz="0.0 0.0 0.0" rpy="0.0 0.0 0.0" />
+  </joint>
+  <xacro:include filename="$(find motoman_sda10f_support)/urdf/sda10f_macro.xacro" />
+  <!-- <xacro:motoman_sda10f prefix=""/> -->
+  <xacro:include filename="$(find motoman_sda10f_support)/urdf/sda10f_transmission.xacro"/>
+  <xacro:include filename="$(find motoman_sda10f_support)/urdf/gazebo_plugin.xacro"/>
 </robot>

Commit message: Squashed changes from ef92997 to 03a3fc4

File: motoman_sda10f_support/urdf/arm_macro.xacro (robot description, xacro)
@@ -1,5 +1,14 @@
 <?xml version="1.0" ?>
 <robot xmlns:xacro="http://ros.org/wiki/xacro">
-	<xacro:macro name="motoman_arm" params="name prefix parent *origin reflect">
+	<xacro:macro name="motoman_arm" params="name prefix parent *origin reflect
+		joint_limited
+		link_1_s_lower_limit:=${-pi}  link_1_s_upper_limit:=${pi}
+        link_2_l_lower_limit:=${-pi}  link_2_l_upper_limit:=${pi}
+        link_3_e_lower_limit:=${-pi}  link_3_e_upper_limit:=${pi}
+        link_4_u_lower_limit:=${-pi}  link_4_u_upper_limit:=${pi}
+        link_5_r_lower_limit:=${-pi}  link_5_r_upper_limit:=${pi}
+        link_6_b_lower_limit:=${-pi}  link_6_b_upper_limit:=${pi}
+        link_7_t_lower_limit:=${-pi}  link_7_t_upper_limit:=${pi}
+        ">
 		<link name="${prefix}link_1_s">
 			<visual>
@@ -19,4 +28,10 @@
 				<material name="yellow"/>
 			</collision>
+	    <inertial>
+	      <mass value="1" />
+	      <inertia ixx="1.0" ixy="0.0" ixz="0.0"
+	               iyy="1.0" iyz="0.0"
+	               izz="1.0" />
+	    </inertial>
 		</link>
 		<link name="${prefix}link_2_l">
@@ -35,4 +50,10 @@
 				<material name="yellow"/>
 			</collision>
+	    <inertial>
+	      <mass value="1" />
+	      <inertia ixx="1.0" ixy="0.0" ixz="0.0"
+	               iyy="1.0" iyz="0.0"
+	               izz="1.0" />
+	    </inertial>
 		</link>
 		<link name="${prefix}link_3_e">
@@ -51,4 +72,10 @@
 				<material name="yellow"/>
 			</collision>
+	    <inertial>
+	      <mass value="1" />
+	      <inertia ixx="1.0" ixy="0.0" ixz="0.0"
+	               iyy="1.0" iyz="0.0"
+	               izz="1.0" />
+	    </inertial>
 		</link>
 		<link name="${prefix}link_4_u">
@@ -67,4 +94,10 @@
 				<material name="yellow"/>
 			</collision>
+	    <inertial>
+	      <mass value="1" />
+	      <inertia ixx="1.0" ixy="0.0" ixz="0.0"
+	               iyy="1.0" iyz="0.0"
+	               izz="1.0" />
+	    </inertial>
 		</link>
 		<link name="${prefix}link_5_r">
@@ -83,4 +116,10 @@
 				<material name="yellow"/>
 			</collision>
+	    <inertial>
+	      <mass value="1" />
+	      <inertia ixx="1.0" ixy="0.0" ixz="0.0"
+	               iyy="1.0" iyz="0.0"
+	               izz="1.0" />
+	    </inertial>
 		</link>
 		<link name="${prefix}link_6_b">
@@ -99,4 +138,10 @@
 				<material name="yellow"/>
 			</collision>
+	    <inertial>
+	      <mass value="1" />
+	      <inertia ixx="1.0" ixy="0.0" ixz="0.0"
+	               iyy="1.0" iyz="0.0"
+	               izz="1.0" />
+	    </inertial>
 		</link>
 		<link name="${prefix}link_7_t">
@@ -113,6 +158,19 @@
 				<material name="yellow"/>
 			</collision>
-		</link>
-	    <link name="${prefix}link_tool0" />
+	    <inertial>
+	      <mass value="1" />
+	      <inertia ixx="1.0" ixy="0.0" ixz="0.0"
+	               iyy="1.0" iyz="0.0"
+	               izz="1.0" />
+	    </inertial>
+		</link>
+	    <link name="${prefix}link_tool0" >
+	    <inertial>
+	      <mass value="1" />
+	      <inertia ixx="1.0" ixy="0.0" ixz="0.0"
+	               iyy="1.0" iyz="0.0"
+	               izz="1.0" />
+	    </inertial>
+</link>
 		<joint name="${prefix}joint_1_s" type="revolute">
 			<parent link="${parent}"/>
@@ -120,5 +178,10 @@
 			<origin xyz="0.09996 ${reflect*0.0275} 0.32214" rpy="1.57 0 ${(reflect-1)*1.57}"/>
 			<axis xyz="0 0 ${-reflect}" />
-			<limit lower="-3.13" upper="3.13" effort="0" velocity="2.95" />
+			<xacro:unless value="${joint_limited}">
+				<limit lower="-3.13" upper="3.13" effort="0" velocity="2.95" />
+			</xacro:unless>
+            <xacro:if value="${joint_limited}">
+            	<limit lower="${link_1_s_lower_limit}" upper="${link_1_s_upper_limit}" effort="150.0" velocity="3.15"/>
+			</xacro:if>
 		</joint>
 		<joint name="${prefix}joint_2_l" type="revolute">
@@ -127,5 +190,10 @@
 			<origin xyz="0 0.0577 -0.2255" rpy="-1.57 0 0"/>
 			<axis xyz="0 0 ${-reflect}" />
-			<limit lower="-1.90" upper="1.90" effort="0" velocity="2.95" />
+			<xacro:unless value="${joint_limited}">
+			    <limit lower="-1.90" upper="1.90" effort="0" velocity="2.95" />
+			</xacro:unless>
+			<xacro:if value="${joint_limited}">
+            	<limit lower="${link_2_l_lower_limit}" upper="${link_2_l_upper_limit}" effort="150.0" velocity="3.15"/>
+			</xacro:if>
 		</joint>
 		<joint name="${prefix}joint_3_e" type="revolute">
@@ -134,5 +202,10 @@
 			<origin xyz="0 0.1690 -0.0454" rpy="1.57 0 0"/>
 			<axis xyz="0 0 ${-reflect}" />
-			<limit lower="-2.95" upper="2.95" effort="0" velocity="2.95" />
+			<xacro:unless value="${joint_limited}">
+				<limit lower="-2.95" upper="2.95" effort="0" velocity="2.95" />
+			</xacro:unless>
+			<xacro:if value="${joint_limited}">
+            	<limit lower="${link_3_e_lower_limit}" upper="${link_3_e_upper_limit}" effort="150.0" velocity="3.15"/>
+			</xacro:if>
 		</joint>
 		<joint name="${prefix}joint_4_u" type="revolute">
@@ -141,5 +214,10 @@
 			<origin xyz="0 -0.0085 -0.181" rpy="-1.57 0 0"/>
 			<axis xyz="0 0 ${reflect}" />
-			<limit lower="-2.36" upper="2.36" effort="0" velocity="2.95" />
+			<xacro:unless value="${joint_limited}">
+				<limit lower="-2.36" upper="2.36" effort="0" velocity="2.95" />
+			</xacro:unless>
+			<xacro:if value="${joint_limited}">
+            	<limit lower="${link_4_u_lower_limit}" upper="${link_4_u_upper_limit}" effort="150.0" velocity="3.15"/>
+			</xacro:if>
 		</joint>
 		<joint name="${prefix}joint_5_r" type="revolute">
@@ -148,5 +226,10 @@
 			<origin xyz="0 0.1936 0.0155" rpy="1.57 0 0"/>
 			<axis xyz="0 0 ${reflect}" />
-			<limit lower="-3.13" upper="3.13" effort="0" velocity="3.48" />
+			<xacro:unless value="${joint_limited}">
+				<limit lower="-3.13" upper="3.13" effort="0" velocity="3.48" />
+			</xacro:unless>
+			<xacro:if value="${joint_limited}">
+            	<limit lower="${link_5_r_lower_limit}" upper="${link_5_r_upper_limit}" effort="150.0" velocity="3.15"/>
+			</xacro:if>
 		</joint>
 		<joint name="${prefix}joint_6_b" type="revolute">
@@ -155,5 +238,10 @@
 			<origin xyz="0 0.0080 -0.155" rpy="-1.57 0 0"/>
 			<axis xyz="0 0 ${reflect}" />
-			<limit lower="-1.90" upper="1.90" effort="0" velocity="3.48" />
+			<xacro:unless value="${joint_limited}">
+				<limit lower="-1.90" upper="1.90" effort="0" velocity="3.48" />
+			</xacro:unless>
+			<xacro:if value="${joint_limited}">
+            	<limit lower="${link_6_b_lower_limit}" upper="${link_6_b_upper_limit}" effort="150.0" velocity="3.15"/>
+			</xacro:if>
 		</joint>
 		<joint name="${prefix}joint_7_t" type="revolute">
@@ -162,5 +250,10 @@
 			<origin xyz="0 0.168 -0.015" rpy="1.57 0 0"/>
 			<axis xyz="0 0 ${-reflect}" />
-			<limit lower="-3.13" upper="3.13" effort="0" velocity="6.97" />
+			<xacro:unless value="${joint_limited}">
+				<limit lower="-3.13" upper="3.13" effort="0" velocity="6.97" />
+			</xacro:unless>
+			<xacro:if value="${joint_limited}">
+            	<limit lower="${link_7_t_lower_limit}" upper="${link_7_t_upper_limit}" effort="150.0" velocity="3.15"/>
+			</xacro:if>
 		</joint>
     <joint name="${prefix}joint_tool0" type="fixed" >

File: motoman_sda10f_support/urdf/common_torso_macro.xacro (robot description, xacro)
@@ -20,4 +20,10 @@
 				</material>
 			</collision>
+	    <inertial>
+	      <mass value="1" />
+	      <inertia ixx="1.0" ixy="0.0" ixz="0.0"
+	               iyy="1.0" iyz="0.0"
+	               izz="1.0" />
+	    </inertial>
 		</link>
 		<link name="${prefix}link_b1">
@@ -38,6 +44,12 @@
 				<material name="yellow"/>
 			</collision>
+	    <inertial>
+	      <mass value="1" />
+	      <inertia ixx="1.0" ixy="0.0" ixz="0.0"
+	               iyy="1.0" iyz="0.0"
+	               izz="1.0" />
+	    </inertial>
 		</link>
-		<link name="${prefix}link_b2">
+<!-- 		<link name="${prefix}link_b2">
 			<visual>
 				<origin rpy="0 0 0" xyz="0 0 0"/>
@@ -56,5 +68,11 @@
 				<material name="yellow"/>
 			</collision>
-		</link>
+	    <inertial>
+	      <mass value="1" />
+	      <inertia ixx="1.0" ixy="0.0" ixz="0.0"
+	               iyy="1.0" iyz="0.0"
+	               izz="1.0" />
+	    </inertial>
+		</link> -->
 		<!-- joint list -->
 		<joint name="${prefix}joint_b1" type="revolute">
@@ -65,6 +83,6 @@
 			<limit lower="-2.9570" upper="2.9570" effort="100" velocity="2.26" />
 		</joint>
-		<joint name="${prefix}joint_b2" type="revolute">
-			<parent link="${prefix}base_link"/>
+<!-- 		<joint name="${prefix}joint_b2" type="revolute">
+			<parent link="base_link"/>
 			<child link="${prefix}link_b2"/>
 			<origin xyz="0.09257 0 0.8835" rpy="0 0 0"/>
@@ -72,5 +90,5 @@
 			<limit lower="-2.9570" upper="2.9570" effort="100" velocity="2.26" />
 			<mimic joint="${prefix}joint_b1" multiplier="1" offset="0"/>
-		</joint>
+		</joint> -->
 		<!-- end of joint list -->
 	</xacro:macro>

File: motoman_sda10f_support/urdf/sda10f_joint_limited.xacro (robot description, xacro)
@@ -7,5 +7,5 @@
     <origin xyz="0.0 0.0 0.0" rpy="0.0 0.0 0.0" />
   </joint>
-  <xacro:include filename="$(find motoman_sda10f_support)/urdf/sda10f_macro.xacro" />
+  <xacro:include filename="$(find motoman_sda10f_support)/urdf/sda10f_joint_limited_macro.xacro" />
   <!-- <xacro:motoman_sda10f prefix=""/> -->
   <xacro:include filename="$(find motoman_sda10f_support)/urdf/sda10f_transmission.xacro"/>

Commit message: add posibility to limit joints

File: motoman_sda10f_support/urdf/arm_macro.xacro (robot description, xacro)
@@ -1,5 +1,14 @@
 <?xml version="1.0" ?>
 <robot xmlns:xacro="http://ros.org/wiki/xacro">
-	<xacro:macro name="motoman_arm" params="name prefix parent *origin reflect">
+	<xacro:macro name="motoman_arm" params="name prefix parent *origin reflect
+		joint_limited
+		link_1_s_lower_limit:=${-pi}  link_1_s_upper_limit:=${pi}
+        link_2_l_lower_limit:=${-pi}  link_2_l_upper_limit:=${pi}
+        link_3_e_lower_limit:=${-pi}  link_3_e_upper_limit:=${pi}
+        link_4_u_lower_limit:=${-pi}  link_4_u_upper_limit:=${pi}
+        link_5_r_lower_limit:=${-pi}  link_5_r_upper_limit:=${pi}
+        link_6_b_lower_limit:=${-pi}  link_6_b_upper_limit:=${pi}
+        link_7_t_lower_limit:=${-pi}  link_7_t_upper_limit:=${pi}
+        ">
 		<link name="${prefix}link_1_s">
 			<visual>
@@ -169,5 +178,10 @@
 			<origin xyz="0.09996 ${reflect*0.0275} 0.32214" rpy="1.57 0 ${(reflect-1)*1.57}"/>
 			<axis xyz="0 0 ${-reflect}" />
-			<limit lower="-3.13" upper="3.13" effort="0" velocity="2.95" />
+			<xacro:unless value="${joint_limited}">
+				<limit lower="-3.13" upper="3.13" effort="0" velocity="2.95" />
+			</xacro:unless>
+            <xacro:if value="${joint_limited}">
+            	<limit lower="${link_1_s_lower_limit}" upper="${link_1_s_upper_limit}" effort="150.0" velocity="3.15"/>
+			</xacro:if>
 		</joint>
 		<joint name="${prefix}joint_2_l" type="revolute">
@@ -176,5 +190,10 @@
 			<origin xyz="0 0.0577 -0.2255" rpy="-1.57 0 0"/>
 			<axis xyz="0 0 ${-reflect}" />
-			<limit lower="-1.90" upper="1.90" effort="0" velocity="2.95" />
+			<xacro:unless value="${joint_limited}">
+			    <limit lower="-1.90" upper="1.90" effort="0" velocity="2.95" />
+			</xacro:unless>
+			<xacro:if value="${joint_limited}">
+            	<limit lower="${link_2_l_lower_limit}" upper="${link_2_l_upper_limit}" effort="150.0" velocity="3.15"/>
+			</xacro:if>
 		</joint>
 		<joint name="${prefix}joint_3_e" type="revolute">
@@ -183,5 +202,10 @@
 			<origin xyz="0 0.1690 -0.0454" rpy="1.57 0 0"/>
 			<axis xyz="0 0 ${-reflect}" />
-			<limit lower="-2.95" upper="2.95" effort="0" velocity="2.95" />
+			<xacro:unless value="${joint_limited}">
+				<limit lower="-2.95" upper="2.95" effort="0" velocity="2.95" />
+			</xacro:unless>
+			<xacro:if value="${joint_limited}">
+            	<limit lower="${link_3_e_lower_limit}" upper="${link_3_e_upper_limit}" effort="150.0" velocity="3.15"/>
+			</xacro:if>
 		</joint>
 		<joint name="${prefix}joint_4_u" type="revolute">
@@ -190,5 +214,10 @@
 			<origin xyz="0 -0.0085 -0.181" rpy="-1.57 0 0"/>
 			<axis xyz="0 0 ${reflect}" />
-			<limit lower="-2.36" upper="2.36" effort="0" velocity="2.95" />
+			<xacro:unless value="${joint_limited}">
+				<limit lower="-2.36" upper="2.36" effort="0" velocity="2.95" />
+			</xacro:unless>
+			<xacro:if value="${joint_limited}">
+            	<limit lower="${link_4_u_lower_limit}" upper="${link_4_u_upper_limit}" effort="150.0" velocity="3.15"/>
+			</xacro:if>
 		</joint>
 		<joint name="${prefix}joint_5_r" type="revolute">
@@ -197,5 +226,10 @@
 			<origin xyz="0 0.1936 0.0155" rpy="1.57 0 0"/>
 			<axis xyz="0 0 ${reflect}" />
-			<limit lower="-3.13" upper="3.13" effort="0" velocity="3.48" />
+			<xacro:unless value="${joint_limited}">
+				<limit lower="-3.13" upper="3.13" effort="0" velocity="3.48" />
+			</xacro:unless>
+			<xacro:if value="${joint_limited}">
+            	<limit lower="${link_5_r_lower_limit}" upper="${link_5_r_upper_limit}" effort="150.0" velocity="3.15"/>
+			</xacro:if>
 		</joint>
 		<joint name="${prefix}joint_6_b" type="revolute">
@@ -204,5 +238,10 @@
 			<origin xyz="0 0.0080 -0.155" rpy="-1.57 0 0"/>
 			<axis xyz="0 0 ${reflect}" />
-			<limit lower="-1.90" upper="1.90" effort="0" velocity="3.48" />
+			<xacro:unless value="${joint_limited}">
+				<limit lower="-1.90" upper="1.90" effort="0" velocity="3.48" />
+			</xacro:unless>
+			<xacro:if value="${joint_limited}">
+            	<limit lower="${link_6_b_lower_limit}" upper="${link_6_b_upper_limit}" effort="150.0" velocity="3.15"/>
+			</xacro:if>
 		</joint>
 		<joint name="${prefix}joint_7_t" type="revolute">
@@ -211,5 +250,10 @@
 			<origin xyz="0 0.168 -0.015" rpy="1.57 0 0"/>
 			<axis xyz="0 0 ${-reflect}" />
-			<limit lower="-3.13" upper="3.13" effort="0" velocity="6.97" />
+			<xacro:unless value="${joint_limited}">
+				<limit lower="-3.13" upper="3.13" effort="0" velocity="6.97" />
+			</xacro:unless>
+			<xacro:if value="${joint_limited}">
+            	<limit lower="${link_7_t_lower_limit}" upper="${link_7_t_upper_limit}" effort="150.0" velocity="3.15"/>
+			</xacro:if>
 		</joint>
     <joint name="${prefix}joint_tool0" type="fixed" >

File: motoman_sda10f_support/urdf/sda10f_macro.xacro (robot description, xacro)
@@ -5,8 +5,10 @@
         <xacro:include filename="$(find motoman_sda10f_support)/urdf/arm_macro.xacro" />
         <xacro:torso name="torso" prefix="torso_"/>
-        <xacro:motoman_arm name="arm_left" prefix="arm_left_" parent="torso_link_b1" reflect="1">
+        <xacro:property name="pi" value="3.1415926535897931"/>
+        <xacro:property name="pi_2" value="1.5707963267948966"/>
+        <xacro:motoman_arm name="arm_left" prefix="arm_left_" parent="torso_link_b1" reflect="1" joint_limited="false">
             <origin xyz="0.09996 0.0275 0.32214" rpy="1.57 0 0" />
         </xacro:motoman_arm>
-        <xacro:motoman_arm name="arm_right" prefix="arm_right_" parent="torso_link_b1" reflect="-1">
+        <xacro:motoman_arm name="arm_right" prefix="arm_right_" parent="torso_link_b1" reflect="-1" joint_limited="false">
             <origin xyz="0.09996 -0.0275 0.32214" rpy="1.57 0 0" />
         </xacro:motoman_arm>

Commit message: set joints velocity and effort limits to original values

File: motoman_sda10f_support/urdf/arm_macro.xacro (robot description, xacro)
@@ -181,6 +181,6 @@
 				<limit lower="-3.13" upper="3.13" effort="0" velocity="2.95" />
 			</xacro:unless>
-            <xacro:if value="${joint_limited}">
-            	<limit lower="${link_1_s_lower_limit}" upper="${link_1_s_upper_limit}" effort="150.0" velocity="3.15"/>
+      <xacro:if value="${joint_limited}">
+        <limit lower="${link_1_s_lower_limit}" upper="${link_1_s_upper_limit}" effort="0" velocity="2.95"/>
 			</xacro:if>
 		</joint>
@@ -194,5 +194,5 @@
 			</xacro:unless>
 			<xacro:if value="${joint_limited}">
-            	<limit lower="${link_2_l_lower_limit}" upper="${link_2_l_upper_limit}" effort="150.0" velocity="3.15"/>
+        <limit lower="${link_2_l_lower_limit}" upper="${link_2_l_upper_limit}" effort="0" velocity="2.95"/>
 			</xacro:if>
 		</joint>
@@ -206,5 +206,5 @@
 			</xacro:unless>
 			<xacro:if value="${joint_limited}">
-            	<limit lower="${link_3_e_lower_limit}" upper="${link_3_e_upper_limit}" effort="150.0" velocity="3.15"/>
+        <limit lower="${link_3_e_lower_limit}" upper="${link_3_e_upper_limit}" effort="0" velocity="2.95"/>
 			</xacro:if>
 		</joint>
@@ -218,5 +218,5 @@
 			</xacro:unless>
 			<xacro:if value="${joint_limited}">
-            	<limit lower="${link_4_u_lower_limit}" upper="${link_4_u_upper_limit}" effort="150.0" velocity="3.15"/>
+        <limit lower="${link_4_u_lower_limit}" upper="${link_4_u_upper_limit}" effort="0" velocity="2.95"/>
 			</xacro:if>
 		</joint>
@@ -230,5 +230,5 @@
 			</xacro:unless>
 			<xacro:if value="${joint_limited}">
-            	<limit lower="${link_5_r_lower_limit}" upper="${link_5_r_upper_limit}" effort="150.0" velocity="3.15"/>
+        <limit lower="${link_5_r_lower_limit}" upper="${link_5_r_upper_limit}" effort="0" velocity="3.48"/>
 			</xacro:if>
 		</joint>
@@ -242,5 +242,5 @@
 			</xacro:unless>
 			<xacro:if value="${joint_limited}">
-            	<limit lower="${link_6_b_lower_limit}" upper="${link_6_b_upper_limit}" effort="150.0" velocity="3.15"/>
+        <limit lower="${link_6_b_lower_limit}" upper="${link_6_b_upper_limit}" effort="0" velocity="3.48"/>
 			</xacro:if>
 		</joint>
@@ -254,5 +254,5 @@
 			</xacro:unless>
 			<xacro:if value="${joint_limited}">
-            	<limit lower="${link_7_t_lower_limit}" upper="${link_7_t_upper_limit}" effort="150.0" velocity="3.15"/>
+        <limit lower="${link_7_t_lower_limit}" upper="${link_7_t_upper_limit}" effort="0" velocity="6.97"/>
 			</xacro:if>
 		</joint>

Commit message: invert rotation sign of sda10f joint_7t

File: motoman_sda10f_support/urdf/arm_macro.xacro (robot description, xacro)
@@ -248,5 +248,5 @@
 			<parent link="${prefix}link_6_b"/>
 			<child link="${prefix}link_7_t"/>
-			<origin xyz="0 0.168 -0.015" rpy="1.57 0 0"/>
+			<origin xyz="0 0.168 -0.015" rpy="-1.57 0 0"/>
 			<axis xyz="0 0 ${-reflect}" />
 			<xacro:unless value="${joint_limited}">
