Commit message: add geometrical calibration for let arm

File: motoman_sda10f_support/urdf/arm_macro.xacro (robot description, xacro)
@@ -3,4 +3,53 @@
 	<xacro:macro name="motoman_arm" params="name prefix parent *origin reflect
 		joint_limited
+		joint_1_s_joint_offset:=${0.0}
+		joint_2_l_joint_offset:=${0.0}
+		joint_3_e_joint_offset:=${0.0}
+		joint_4_u_joint_offset:=${0.0}
+		joint_5_r_joint_offset:=${0.0}
+		joint_6_b_joint_offset:=${0.0}
+		joint_7_t_joint_offset:=${0.0}
+		joint_1_s_joint_x_offset:=${0.0}
+		joint_1_s_joint_y_offset:=${0.0}
+		joint_1_s_joint_z_offset:=${0.0}
+		joint_1_s_joint_a_offset:=${0.0}
+		joint_1_s_joint_b_offset:=${0.0}
+		joint_1_s_joint_c_offset:=${0.0}
+		joint_2_l_joint_x_offset:=${0.0}
+		joint_2_l_joint_y_offset:=${0.0}
+		joint_2_l_joint_z_offset:=${0.0}
+		joint_2_l_joint_a_offset:=${0.0}
+		joint_2_l_joint_b_offset:=${0.0}
+		joint_2_l_joint_c_offset:=${0.0}
+		joint_3_e_joint_x_offset:=${0.0}
+		joint_3_e_joint_y_offset:=${0.0}
+		joint_3_e_joint_z_offset:=${0.0}
+		joint_3_e_joint_a_offset:=${0.0}
+		joint_3_e_joint_b_offset:=${0.0}
+		joint_3_e_joint_c_offset:=${0.0}
+		joint_4_u_joint_x_offset:=${0.0}
+		joint_4_u_joint_y_offset:=${0.0}
+		joint_4_u_joint_z_offset:=${0.0}
+		joint_4_u_joint_a_offset:=${0.0}
+		joint_4_u_joint_b_offset:=${0.0}
+		joint_4_u_joint_c_offset:=${0.0}
+		joint_5_r_joint_x_offset:=${0.0}
+		joint_5_r_joint_y_offset:=${0.0}
+		joint_5_r_joint_z_offset:=${0.0}
+		joint_5_r_joint_a_offset:=${0.0}
+		joint_5_r_joint_b_offset:=${0.0}
+		joint_5_r_joint_c_offset:=${0.0}
+		joint_6_b_joint_x_offset:=${0.0}
+		joint_6_b_joint_y_offset:=${0.0}
+		joint_6_b_joint_z_offset:=${0.0}
+		joint_6_b_joint_a_offset:=${0.0}
+		joint_6_b_joint_b_offset:=${0.0}
+		joint_6_b_joint_c_offset:=${0.0}
+		joint_7_t_joint_x_offset:=${0.0}
+		joint_7_t_joint_y_offset:=${0.0}
+		joint_7_t_joint_z_offset:=${0.0}
+		joint_7_t_joint_a_offset:=${0.0}
+		joint_7_t_joint_b_offset:=${0.0}
+		joint_7_t_joint_c_offset:=${0.0}
 		link_1_s_lower_limit:=${-pi}  link_1_s_upper_limit:=${pi}
         link_2_l_lower_limit:=${-pi}  link_2_l_upper_limit:=${pi}
@@ -35,4 +84,12 @@
 	    </inertial>
 		</link>
+		<link name="${prefix}2_l_link_offset">
+		<inertial>
+              <mass value="1" />
+              <inertia ixx="1.0" ixy="0.0" ixz="0.0"
+                       iyy="1.0" iyz="0.0"
+                       izz="1.0" />
+        </inertial>
+        </link>
 		<link name="${prefix}link_2_l">
 			<visual>
@@ -57,4 +114,12 @@
 	    </inertial>
 		</link>
+		<link name="${prefix}3_e_link_offset">
+		<inertial>
+              <mass value="1" />
+              <inertia ixx="1.0" ixy="0.0" ixz="0.0"
+                       iyy="1.0" iyz="0.0"
+                       izz="1.0" />
+        </inertial>
+        </link>
 		<link name="${prefix}link_3_e">
 			<visual>
@@ -79,4 +144,12 @@
 	    </inertial>
 		</link>
+		<link name="${prefix}4_u_link_offset">
+		<inertial>
+              <mass value="1" />
+              <inertia ixx="1.0" ixy="0.0" ixz="0.0"
+                       iyy="1.0" iyz="0.0"
+                       izz="1.0" />
+        </inertial>
+        </link>
 		<link name="${prefix}link_4_u">
 			<visual>
@@ -101,4 +174,12 @@
 	    </inertial>
 		</link>
+		<link name="${prefix}5_r_link_offset">
+		<inertial>
+              <mass value="1" />
+              <inertia ixx="1.0" ixy="0.0" ixz="0.0"
+                       iyy="1.0" iyz="0.0"
+                       izz="1.0" />
+        </inertial>
+        </link>
 		<link name="${prefix}link_5_r">
 			<visual>
@@ -123,4 +204,12 @@
 	    </inertial>
 		</link>
+		<link name="${prefix}6_b_link_offset">
+		<inertial>
+              <mass value="1" />
+              <inertia ixx="1.0" ixy="0.0" ixz="0.0"
+                       iyy="1.0" iyz="0.0"
+                       izz="1.0" />
+        </inertial>
+        </link>
 		<link name="${prefix}link_6_b">
 			<visual>
@@ -145,4 +234,12 @@
 	    </inertial>
 		</link>
+		<link name="${prefix}7_t_link_offset">
+		<inertial>
+              <mass value="1" />
+              <inertia ixx="1.0" ixy="0.0" ixz="0.0"
+                       iyy="1.0" iyz="0.0"
+                       izz="1.0" />
+        </inertial>
+        </link>
 		<link name="${prefix}link_7_t">
 			<visual>
@@ -176,5 +273,5 @@
 			<parent link="${parent}"/>
 			<child link="${prefix}link_1_s"/>
-			<origin xyz="0.09996 ${reflect*0.0275} 0.32214" rpy="1.57 0 ${(reflect-1)*1.57}"/>
+			<origin xyz="0.09996 ${reflect*0.0275} 0.32214" rpy="1.57 0 ${(reflect-1)*1.57+joint_1_s_joint_offset}"/>
 			<axis xyz="0 0 ${-reflect}" />
 			<xacro:unless value="${joint_limited}">
@@ -185,8 +282,14 @@
 			</xacro:if>
 		</joint>
+		<joint name="${prefix}2_l_joint_offset" type="fixed">
+			<origin xyz="${joint_2_l_joint_x_offset} ${joint_2_l_joint_y_offset} ${joint_2_l_joint_z_offset}"
+			rpy="${joint_2_l_joint_a_offset} ${joint_2_l_joint_b_offset} ${joint_2_l_joint_c_offset}"/>
+			<parent link="${prefix}link_1_s"/>
+			<child link="${prefix}2_l_link_offset"/>
+		</joint>
 		<joint name="${prefix}joint_2_l" type="revolute">
-			<parent link="${prefix}link_1_s"/>
+			<parent link="${prefix}2_l_link_offset"/>
 			<child link="${prefix}link_2_l"/>
-			<origin xyz="0 0.0577 -0.2255" rpy="-1.57 0 0"/>
+			<origin xyz="0 0.0577 -0.2255" rpy="-1.57 0 ${joint_2_l_joint_offset}"/>
 			<axis xyz="0 0 ${-reflect}" />
 			<xacro:unless value="${joint_limited}">
@@ -197,8 +300,14 @@
 			</xacro:if>
 		</joint>
+		<joint name="${prefix}3_e_joint_offset" type="fixed">
+			<origin xyz="${joint_3_e_joint_x_offset} ${joint_3_e_joint_y_offset} ${joint_3_e_joint_z_offset}"
+			rpy="${joint_3_e_joint_a_offset} ${joint_3_e_joint_b_offset} ${joint_3_e_joint_c_offset}"/>
+			<parent link="${prefix}link_2_l"/>
+			<child link="${prefix}3_e_link_offset"/>
+		</joint>
 		<joint name="${prefix}joint_3_e" type="revolute">
-			<parent link="${prefix}link_2_l"/>
+			<parent link="${prefix}3_e_link_offset"/>
 			<child link="${prefix}link_3_e"/>
-			<origin xyz="0 0.1690 -0.0454" rpy="1.57 0 0"/>
+			<origin xyz="0 0.1690 -0.0454" rpy="1.57 0 ${joint_3_e_joint_offset}"/>
 			<axis xyz="0 0 ${-reflect}" />
 			<xacro:unless value="${joint_limited}">
@@ -209,8 +318,14 @@
 			</xacro:if>
 		</joint>
+		<joint name="${prefix}4_u_joint_offset" type="fixed">
+			<origin xyz="${joint_4_u_joint_x_offset} ${joint_4_u_joint_y_offset} ${joint_4_u_joint_z_offset}"
+			rpy="${joint_4_u_joint_a_offset} ${joint_4_u_joint_b_offset} ${joint_4_u_joint_c_offset}"/>
+			<parent link="${prefix}link_3_e"/>
+			<child link="${prefix}4_u_link_offset"/>
+		</joint>
 		<joint name="${prefix}joint_4_u" type="revolute">
-			<parent link="${prefix}link_3_e"/>
+			<parent link="${prefix}4_u_link_offset"/>
 			<child link="${prefix}link_4_u"/>
-			<origin xyz="0 -0.0085 -0.181" rpy="-1.57 0 0"/>
+			<origin xyz="0 -0.0085 -0.181" rpy="-1.57 0 ${joint_4_u_joint_offset}"/>
 			<axis xyz="0 0 ${reflect}" />
 			<xacro:unless value="${joint_limited}">
@@ -221,8 +336,14 @@
 			</xacro:if>
 		</joint>
+		<joint name="${prefix}5_r_joint_offset" type="fixed">
+			<origin xyz="${joint_5_r_joint_x_offset} ${joint_5_r_joint_y_offset} ${joint_5_r_joint_z_offset}"
+			rpy="${joint_5_r_joint_a_offset} ${joint_5_r_joint_b_offset} ${joint_5_r_joint_c_offset}"/>
+			<parent link="${prefix}link_4_u"/>
+			<child link="${prefix}5_r_link_offset"/>
+		</joint>
 		<joint name="${prefix}joint_5_r" type="revolute">
-			<parent link="${prefix}link_4_u"/>
+			<parent link="${prefix}5_r_link_offset"/>
 			<child link="${prefix}link_5_r"/>
-			<origin xyz="0 0.1936 0.0155" rpy="1.57 0 0"/>
+			<origin xyz="0 0.1936 0.0155" rpy="1.57 0 ${joint_5_r_joint_offset}"/>
 			<axis xyz="0 0 ${reflect}" />
 			<xacro:unless value="${joint_limited}">
@@ -233,8 +354,14 @@
 			</xacro:if>
 		</joint>
+		<joint name="${prefix}6_b_joint_offset" type="fixed">
+			<origin xyz="${joint_6_b_joint_x_offset} ${joint_6_b_joint_y_offset} ${joint_6_b_joint_z_offset}"
+			rpy="${joint_6_b_joint_a_offset} ${joint_6_b_joint_b_offset} ${joint_6_b_joint_c_offset}"/>
+			<parent link="${prefix}link_5_r"/>
+			<child link="${prefix}6_b_link_offset"/>
+		</joint>
 		<joint name="${prefix}joint_6_b" type="revolute">
-			<parent link="${prefix}link_5_r"/>
+			<parent link="${prefix}6_b_link_offset"/>
 			<child link="${prefix}link_6_b"/>
-			<origin xyz="0 0.0080 -0.155" rpy="-1.57 0 0"/>
+			<origin xyz="0 0.0080 -0.155" rpy="-1.57 0 ${joint_6_b_joint_offset}"/>
 			<axis xyz="0 0 ${reflect}" />
 			<xacro:unless value="${joint_limited}">
@@ -245,8 +372,14 @@
 			</xacro:if>
 		</joint>
+		<joint name="${prefix}7_t_joint_offset" type="fixed">
+			<origin xyz="${joint_7_t_joint_x_offset} ${joint_7_t_joint_y_offset} ${joint_7_t_joint_z_offset}"
+			rpy="${joint_7_t_joint_a_offset} ${joint_7_t_joint_b_offset} ${joint_7_t_joint_c_offset}"/>
+			<parent link="${prefix}link_6_b"/>
+			<child link="${prefix}7_t_link_offset"/>
+		</joint>
 		<joint name="${prefix}joint_7_t" type="revolute">
-			<parent link="${prefix}link_6_b"/>
+			<parent link="${prefix}7_t_link_offset"/>
 			<child link="${prefix}link_7_t"/>
-			<origin xyz="0 0.168 -0.015" rpy="-1.57 0 0"/>
+			<origin xyz="0 0.168 -0.015" rpy="-1.57 0 ${joint_7_t_joint_offset}"/>
 			<axis xyz="0 0 ${-reflect}" />
 			<xacro:unless value="${joint_limited}">

File: motoman_sda10f_support/urdf/common_torso_macro.xacro (robot description, xacro)
@@ -1,5 +1,15 @@
 <?xml version="1.0" ?>
 <robot xmlns:xacro="http://ros.org/wiki/xacro">
-	<xacro:macro name="torso" params="name prefix">
+	<xacro:macro name="torso" params="
+		name
+		prefix
+		use_sim
+		torso_joint_b1_joint_offset
+		torso_joint_b1_joint_x_offset
+		torso_joint_b1_joint_y_offset
+		torso_joint_b1_joint_z_offset
+		torso_joint_b1_joint_a_offset
+		torso_joint_b1_joint_b_offset
+		torso_joint_b1_joint_c_offset">
 		<!-- link list -->
 		<link name="${prefix}base_link">
@@ -27,4 +37,12 @@
 	    </inertial>
 		</link>
+		<link name="${prefix}b1_link_offset">
+    	<inertial>
+        	<mass value="1" />
+        	<inertia ixx="1.0" ixy="0.0" ixz="0.0"
+                 iyy="1.0" iyz="0.0"
+                 izz="1.0" />
+      		</inertial>
+    	</link>
 		<link name="${prefix}link_b1">
 			<visual>
@@ -51,44 +69,54 @@
 	    </inertial>
 		</link>
-<!-- 		<link name="${prefix}link_b2">
-			<visual>
-				<origin rpy="0 0 0" xyz="0 0 0"/>
-				<geometry>
-					<mesh filename="package://motoman_sda10f_support/meshes/sda10f/visual/motoman_axis_b1.stl"/>
-				</geometry>
-				<material name="silver">
-					<color rgba="0.8 0.8 0.8 1"/>
-				</material>
-			</visual>
-			<collision>
-				<origin rpy="0 0 0" xyz="0 0 0"/>
-				<geometry>
-					<mesh filename="package://motoman_sda10f_support/meshes/sda10f/collision/motoman_axis_b1.stl" />
-				</geometry>
-				<material name="yellow"/>
-			</collision>
-	    <inertial>
-	      <mass value="1" />
-	      <inertia ixx="1.0" ixy="0.0" ixz="0.0"
-	               iyy="1.0" iyz="0.0"
-	               izz="1.0" />
-	    </inertial>
-		</link> -->
+		<xacro:if value="${use_sim== 'false'}">
+			<link name="${prefix}link_b2">
+				<visual>
+					<origin rpy="0 0 0" xyz="0 0 0"/>
+					<geometry>
+						<mesh filename="package://motoman_sda10f_support/meshes/sda10f/visual/motoman_axis_b1.stl"/>
+					</geometry>
+					<material name="silver">
+						<color rgba="0.8 0.8 0.8 1"/>
+					</material>
+				</visual>
+				<collision>
+					<origin rpy="0 0 0" xyz="0 0 0"/>
+					<geometry>
+						<mesh filename="package://motoman_sda10f_support/meshes/sda10f/collision/motoman_axis_b1.stl" />
+					</geometry>
+					<material name="yellow"/>
+				</collision>
+	    	<inertial>
+	    	  <mass value="1" />
+	    	  <inertia ixx="1.0" ixy="0.0" ixz="0.0"
+	    	           iyy="1.0" iyz="0.0"
+	    	           izz="1.0" />
+	    	</inertial>
+			</link>
+		</xacro:if>
 		<!-- joint list -->
+		<joint name="${prefix}b1_joint_offset" type="fixed">
+			<origin xyz="${torso_joint_b1_joint_x_offset} ${torso_joint_b1_joint_y_offset} ${torso_joint_b1_joint_z_offset}"
+			rpy="${torso_joint_b1_joint_a_offset} ${torso_joint_b1_joint_b_offset} ${torso_joint_b1_joint_c_offset}"/>
+			<parent link="${prefix}base_link"/>
+			<child link="${prefix}b1_link_offset"/>
+		</joint>
 		<joint name="${prefix}joint_b1" type="revolute">
-			<parent link="${prefix}base_link"/>
+			<parent link="${prefix}b1_link_offset"/>
 			<child link="${prefix}link_b1"/>
-			<origin xyz="0.09257 0 0.8835" rpy="0 0 0"/>
+			<origin xyz="0.09257 0 0.8835" rpy="0 0 ${torso_joint_b1_joint_offset}"/>
 			<axis xyz="0 0 1" />
 			<limit lower="-2.9570" upper="2.9570" effort="100" velocity="2.26" />
 		</joint>
-<!-- 		<joint name="${prefix}joint_b2" type="revolute">
-			<parent link="base_link"/>
-			<child link="${prefix}link_b2"/>
-			<origin xyz="0.09257 0 0.8835" rpy="0 0 0"/>
-			<axis xyz="0 0 1" />
-			<limit lower="-2.9570" upper="2.9570" effort="100" velocity="2.26" />
-			<mimic joint="${prefix}joint_b1" multiplier="1" offset="0"/>
-		</joint> -->
+		<xacro:if value="${use_sim == 'false'}">
+			<joint  if="${use_sim}" name="${prefix}joint_b2" type="revolute">
+				<parent link="${prefix}b1_link_offset"/>
+				<child link="${prefix}link_b2"/>
+				<origin xyz="0.09257 0 0.8835" rpy="0 0  ${torso_joint_b1_joint_offset}"/>
+				<axis xyz="0 0 1" />
+				<limit lower="-2.9570" upper="2.9570" effort="100" velocity="2.26" />
+				<mimic joint="${prefix}joint_b1" multiplier="1" offset="0"/>
+			</joint>
+		</xacro:if>
 		<!-- end of joint list -->
 	</xacro:macro>

File: motoman_sda10f_support/urdf/sda10f.xacro (robot description, xacro)
@@ -8,5 +8,5 @@
   </joint>
   <xacro:include filename="$(find motoman_sda10f_support)/urdf/sda10f_macro.xacro" />
-  <xacro:motoman_sda10f prefix=""/>
+  <xacro:motoman_sda10f prefix="" use_sim="false"/>
   <xacro:include filename="$(find motoman_sda10f_support)/urdf/sda10f_transmission.xacro"/>
   <xacro:include filename="$(find motoman_sda10f_support)/urdf/gazebo_plugin.xacro"/>

File: motoman_sda10f_support/urdf/sda10f_joint_limited.xacro (robot description, xacro)
@@ -8,5 +8,5 @@
   </joint>
   <xacro:include filename="$(find motoman_sda10f_support)/urdf/sda10f_joint_limited_macro.xacro" />
-  <xacro:motoman_sda10f prefix=""/>
+  <xacro:motoman_sda10f prefix="" use_sim="false"/>
   <xacro:include filename="$(find motoman_sda10f_support)/urdf/sda10f_transmission.xacro"/>
   <xacro:include filename="$(find motoman_sda10f_support)/urdf/gazebo_plugin.xacro"/>
