Commit message: update urdf with  official 3D CAD model dimensions
update URDF with official 3D model dimensions

aling joint_1 in the center of the robot

update dimensions with more accurate info

File: motoman_sda10f_support/urdf/arm_macro.xacro (robot description, xacro)
@@ -176,5 +176,5 @@
 			<parent link="${parent}"/>
 			<child link="${prefix}link_1_s"/>
-			<origin xyz="0.09996 ${reflect*0.0275} 0.32214" rpy="1.57 0 ${(reflect-1)*1.57}"/>
+			<origin xyz="0.100 ${reflect*0.0275} 0.3114" rpy="1.57 0 ${(reflect-1)*1.57}"/>
 			<axis xyz="0 0 ${-reflect}" />
 			<xacro:unless value="${joint_limited}">
@@ -188,5 +188,5 @@
 			<parent link="${prefix}link_1_s"/>
 			<child link="${prefix}link_2_l"/>
-			<origin xyz="0 0.0577 -0.2255" rpy="-1.57 0 0"/>
+			<origin xyz="0 0.0539 -0.2375" rpy="-1.57 0 0"/>
 			<axis xyz="0 0 ${-reflect}" />
 			<xacro:unless value="${joint_limited}">
@@ -200,5 +200,5 @@
 			<parent link="${prefix}link_2_l"/>
 			<child link="${prefix}link_3_e"/>
-			<origin xyz="0 0.1690 -0.0454" rpy="1.57 0 0"/>
+			<origin xyz="0 0.211 -0.0539" rpy="1.57 0 0"/>
 			<axis xyz="0 0 ${-reflect}" />
 			<xacro:unless value="${joint_limited}">
@@ -212,5 +212,5 @@
 			<parent link="${prefix}link_3_e"/>
 			<child link="${prefix}link_4_u"/>
-			<origin xyz="0 -0.0085 -0.181" rpy="-1.57 0 0"/>
+			<origin xyz="0 -0.0375 -0.149" rpy="-1.57 0 0"/>
 			<axis xyz="0 0 ${reflect}" />
 			<xacro:unless value="${joint_limited}">
@@ -224,5 +224,5 @@
 			<parent link="${prefix}link_4_u"/>
 			<child link="${prefix}link_5_r"/>
-			<origin xyz="0 0.1936 0.0155" rpy="1.57 0 0"/>
+			<origin xyz="0 0.233 0.0375" rpy="1.57 0 0"/>
 			<axis xyz="0 0 ${reflect}" />
 			<xacro:unless value="${joint_limited}">
@@ -236,5 +236,5 @@
 			<parent link="${prefix}link_5_r"/>
 			<child link="${prefix}link_6_b"/>
-			<origin xyz="0 0.0080 -0.155" rpy="-1.57 0 0"/>
+			<origin xyz="0 0.0335 -0.127" rpy="-1.57 0 0"/>
 			<axis xyz="0 0 ${reflect}" />
 			<xacro:unless value="${joint_limited}">
@@ -248,5 +248,5 @@
 			<parent link="${prefix}link_6_b"/>
 			<child link="${prefix}link_7_t"/>
-			<origin xyz="0 0.168 -0.015" rpy="-1.57 0 0"/>
+			<origin xyz="0 0.155 -0.0335" rpy="-1.57 0 0"/>
 			<axis xyz="0 0 ${-reflect}" />
 			<xacro:unless value="${joint_limited}">

File: motoman_sda10f_support/urdf/sda10f_macro.xacro (robot description, xacro)
@@ -6,8 +6,8 @@
         <xacro:torso name="${prefix}torso" prefix="${prefix}torso_"/>
         <xacro:motoman_arm name="${prefix}arm_left" prefix="${prefix}arm_left_" parent="${prefix}torso_link_b1" reflect="1" joint_limited="false">
-            <origin xyz="0.09996 0.0275 0.32214" rpy="1.57 0 0" />
+            <origin xyz="0.100 0.0275 0.3114" rpy="1.57 0 0" />
         </xacro:motoman_arm>
         <xacro:motoman_arm name="${prefix}arm_right" prefix="${prefix}arm_right_" parent="${prefix}torso_link_b1" reflect="-1" joint_limited="false">
-            <origin xyz="0.09996 -0.0275 0.32214" rpy="1.57 0 0" />
+            <origin xyz="0.100 -0.0275 0.3114" rpy="1.57 0 0" />
         </xacro:motoman_arm>
      </xacro:macro>
